Commit message: feat:  enhanced the Robo Roomba simulation
- Removed debug PDF and GV files related to frame visualizations.
- Updated `cleaning_node.py` to improve PID control logic and state management for the vacuum robot.
- Adjusted CMakeLists.txt to include RViz configuration files.
- Modified `mapper_params_online_async.yaml` to set a minimum laser range for SLAM.
- Enhanced URDF model for the Roomba with improved material properties and added a back caster wheel.
- Updated indoor SDF world file to include a virtual wall and debugging tools for better simulation control.
- Created new navigation parameters in `nav2_params.yaml` for improved robot localization and navigation.
- Added launch files for autonomous mapping and localization, integrating SLAM and navigation functionalities.
- Introduced RViz configuration for better visualization of the robot's environment and sensor data.

File: src/robo_roomba_sim/urdf/roomba.urdf.xacro (robot description, xacro)
@@ -5,5 +5,5 @@
   <!-- ==================================================== -->
   <material name="dark_grey"><color rgba="0.2 0.2 0.2 1"/></material>
-  <material name="light_grey"><color rgba="0.6 0.6 0.6 1"/></material> <!-- Lighter for contrast -->
+  <material name="light_grey"><color rgba="0.6 0.6 0.6 1"/></material>
   <material name="black"><color rgba="0.05 0.05 0.05 1"/></material>
   <material name="blue"><color rgba="0.1 0.1 0.8 1"/></material>
@@ -18,15 +18,11 @@
       <material name="dark_grey"/>
     </visual>
-    <!-- Collision is just the main cylinder -->
     <collision>
       <geometry><cylinder length="0.08" radius="0.17"/></geometry>
     </collision>
-    <!-- 2. The Semicircle Bumper (The Trick) -->
-    <!-- We make a slightly wider cylinder and move it forward -->
+    <!-- 2. Bumper -->
     <visual>
       <origin xyz="0.03 0 0" rpy="0 0 0"/>
       <geometry>
-        <!-- Radius 0.175 is slightly larger than base (0.17) -->
-        <!-- Length 0.06 makes it look like a distinct strip -->
         <cylinder length="0.06" radius="0.175"/>
       </geometry>
@@ -34,5 +30,4 @@
     </visual>
     <!-- 3. Top Decorative Plate -->
-    <!-- Moved UP to z=0.041 to prevent Glitching/Z-Fighting -->
     <visual>
       <origin xyz="0 0 0.041" rpy="0 0 0"/>
@@ -41,5 +36,4 @@
     </visual>
     <!-- 4. Power Button -->
-    <!-- Moved UP to z=0.043 to float above the plate -->
     <visual>
       <origin xyz="-0.05 0 0.043" rpy="0 0 0"/>
@@ -48,6 +42,7 @@
     </visual>
     <inertial>
-      <mass value="3.0"/>
-      <inertia ixx="0.02" ixy="0" ixz="0" iyy="0.02" iyz="0" izz="0.04"/>
+      <mass value="4.0"/>
+      <origin xyz="0 0 -0.02" rpy="0 0 0"/>
+      <inertia ixx="0.03" ixy="0" ixz="0" iyy="0.03" iyz="0" izz="0.06"/>
     </inertial>
   </link>
@@ -63,4 +58,12 @@
     <collision>
       <geometry><cylinder length="0.02" radius="0.033"/></geometry>
+      <surface>
+        <friction>
+          <ode>
+            <mu>1.0</mu>   <!-- High forward friction -->
+            <mu2>0.2</mu2>  <!-- Low sideways friction -->
+          </ode>
+        </friction>
+      </surface>
     </collision>
     <inertial>
@@ -74,4 +77,5 @@
     <origin xyz="0 0.14 -0.025" rpy="-1.57 0 0"/>
     <axis xyz="0 0 1"/>
+    <dynamics damping="0.5" friction="1.0"/>
   </joint>
   <!-- Right Wheel -->
@@ -83,4 +87,12 @@
     <collision>
       <geometry><cylinder length="0.02" radius="0.033"/></geometry>
+      <surface>
+        <friction>
+          <ode>
+            <mu>1.0</mu>
+            <mu2>0.2</mu2>
+          </ode>
+        </friction>
+      </surface>
     </collision>
     <inertial>
@@ -94,7 +106,7 @@
     <origin xyz="0 -0.14 -0.025" rpy="-1.57 0 0"/>
     <axis xyz="0 0 1"/>
-  </joint>
-  <!-- Caster -->
-  <!-- Caster (Ball for balance) -->
+    <dynamics damping="0.5" friction="1.0"/>
+  </joint>
+  <!-- Front Caster Wheel -->
   <link name="caster">
     <visual>
@@ -104,5 +116,4 @@
     <collision>
       <geometry><sphere radius="0.032"/></geometry>
-      <!-- NEW: Low Friction Surface -->
       <surface>
         <friction>
@@ -112,4 +123,10 @@
           </ode>
         </friction>
+        <contact>
+          <ode>
+            <kp>1000000.0</kp>
+            <kd>1.0</kd>
+          </ode>
+        </contact>
       </surface>
     </collision>
@@ -124,4 +141,27 @@
     <origin xyz="0.12 0 -0.025"/>
   </joint>
+  <!-- Back Caster Wheel -->
+  <link name="caster_back">
+    <visual>
+      <geometry><sphere radius="0.032"/></geometry>
+      <material name="black"/>
+    </visual>
+    <collision>
+      <geometry><sphere radius="0.032"/></geometry>
+      <surface>
+        <friction><ode><mu>0.0</mu><mu2>0.0</mu2></ode></friction>
+        <contact><ode><kp>1000000.0</kp><kd>1.0</kd></ode></contact>
+      </surface>
+    </collision>
+    <inertial>
+      <mass value="0.1"/>
+      <inertia ixx="0.001" ixy="0" ixz="0" iyy="0.001" iyz="0" izz="0.001"/>
+    </inertial>
+  </link>
+  <joint name="caster_back_joint" type="fixed">
+    <parent link="base_link"/>
+    <child link="caster_back"/>
+    <origin xyz="-0.12 0 -0.025"/>
+  </joint>
   <!-- ==================================================== -->
   <!-- LIDAR -->
@@ -141,5 +181,4 @@
     <parent link="base_link"/>
     <child link="base_link/lidar"/>
-    <!-- Moved slightly forward to look purposeful -->
     <origin xyz="0.05 0 0.06"/>
   </joint>

Commit message: feat: improve logic on autonomous mapping, added map result, and updated simulation model

File: src/robo_roomba_sim/urdf/roomba.urdf.xacro (robot description, xacro)
@@ -18,6 +18,6 @@
       <material name="dark_grey"/>
     </visual>
-    <collision>
-      <geometry><cylinder length="0.08" radius="0.17"/></geometry>
+    <collision name="base_collision">
+      <geometry><cylinder length="0.08" radius="0.175"/></geometry>
     </collision>
     <!-- 2. Bumper -->
@@ -37,6 +37,6 @@
     <!-- 4. Power Button -->
     <visual>
-      <origin xyz="-0.05 0 0.043" rpy="0 0 0"/>
-      <geometry><cylinder length="0.005" radius="0.015"/></geometry>
+      <origin xyz="-0.05 0 0.05" rpy="0 0 0"/>
+      <geometry><cylinder length="0.01" radius="0.015"/></geometry>
       <material name="green_light"/>
     </visual>
@@ -229,3 +229,13 @@
     </sensor>
   </gazebo>
+  <gazebo reference="base_link">
+    <sensor name="bumper_sensor" type="contact">
+      <always_on>true</always_on>
+      <update_rate>50.0</update_rate>
+      <contact>
+        <collision>base_link_fixed_joint_lump__base_collision_collision</collision>
+      </contact>
+      <topic>bumper</topic>
+    </sensor>
+  </gazebo>
 </robot>
